File: LegoLights/LegoLights.kicad_pcb (KiCad board)
At the start: 2 copper layers, 32 x 8 mm, 4 parts, among them J1 Conn_01x02, J2 Conn_01x02

Commit message: Add icon
Parts:
- added G***: LOGO, Icons:firefly, B.Cu at (141.0, 61.0)
Other:
- board text added: "Lego Lights Rev1.0 rws 2024"
- board text removed: "Lego Lights Rev1.0"
